File: cad/schematic.brd (EAGLE design)
At the start: 47.5 x 32 mm, 28 parts, among them Q1 FC-255, Q2 ISP, U1 74HC595, U2 ATTINY2313, U3 PCA21125

Commit message: wip
Parts:
- added IMG2: SLOT, library:SLOT
Changed lines of the file:
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@@
 <wire x1="45.46" y1="32" x2="2" y2="32" width="0" layer="20"/>
 <wire x1="2" y1="32" x2="0" y2="30" width="0" layer="20" curve="90"/>
-<text x="27.813" y="27.686" size="0.8128" layer="21" font="fixed" rot="R270">MINUTES</text>
+<text x="24.765" y="27.559" size="0.8128" layer="21" font="fixed" rot="R270">MINUTES</text>
 <text x="3.556" y="27.94" size="0.8128" layer="21" font="fixed" rot="R270">HOURS</text>
 <polygon width="0.0005" layer="52" pour="hatch">
@@
 </element>
 <element name="IMG1" library="library" package="IMG6" value="IMAGE" x="-1.905" y="-1.397" smashed="yes"/>
+<element name="IMG2" library="library" package="SLOT" value="SLOT" x="-1.27" y="-11.43" smashed="yes"/>
 </elements>
 <signals>
@@
 <wire x1="17.5" y1="5.33" x2="15.973" y2="5.33" width="0.254" layer="1"/>
 <wire x1="15.973" y1="5.33" x2="15.969" y2="5.334" width="0.254" layer="1"/>
-<wire x1="45.43" y1="12.535" x2="44.107" y2="12.535" width="0.1524" layer="1"/>
-<wire x1="44.107" y1="12.535" x2="43.18" y2="13.462" width="0.1524" layer="1"/>
-<wire x1="43.18" y1="13.462" x2="43.18" y2="22.86" width="0.1524" layer="1"/>
-<wire x1="43.18" y1="22.86" x2="41.91" y2="24.13" width="0.1524" layer="1"/>
-<wire x1="41.91" y1="24.13" x2="39.37" y2="24.13" width="0.1524" layer="1"/>
+<wire x1="45.43" y1="12.535" x2="44.107" y2="12.535" width="0.254" layer="1"/>
+<wire x1="44.107" y1="12.535" x2="43.18" y2="13.462" width="0.254" layer="1"/>
+<wire x1="43.18" y1="13.462" x2="43.18" y2="22.86" width="0.254" layer="1"/>
+<wire x1="43.18" y1="22.86" x2="41.91" y2="24.13" width="0.254" layer="1"/>
+<wire x1="41.91" y1="24.13" x2="39.37" y2="24.13" width="0.254" layer="1"/>
 <via x="39.37" y="24.13" extent="1-16" drill="0.35"/>
-<wire x1="15.969" y1="5.334" x2="15.969" y2="6.002" width="0.1524" layer="1"/>
-<wire x1="14.605" y1="7.366" x2="14.605" y2="7.747" width="0.1524" layer="1"/>
+<wire x1="15.969" y1="5.334" x2="15.969" y2="6.002" width="0.254" layer="1"/>
+<wire x1="14.605" y1="7.366" x2="14.605" y2="7.747" width="0.254" layer="1"/>
 <via x="14.605" y="7.747" extent="1-16" drill="0.35"/>
 <wire x1="14.605" y1="7.747" x2="18.288" y2="11.43" width="0.254" layer="16"/>
@@
 <wire x1="33.02" y1="22.86" x2="34.544" y2="24.384" width="0.254" layer="16"/>
 <wire x1="34.544" y1="24.384" x2="39.37" y2="24.384" width="0.254" layer="16"/>
-<wire x1="15.969" y1="6.002" x2="14.605" y2="7.366" width="0.1524" layer="1"/>
+<wire x1="15.969" y1="6.002" x2="14.605" y2="7.366" width="0.254" layer="1"/>
 <via x="23.368" y="15.494" extent="1-16" drill="0.35"/>
 <wire x1="23.368" y1="15.494" x2="30.734" y2="15.494" width="0.254" layer="16"/>
@@
 <wire x1="18.288" y1="11.43" x2="22.225" y2="11.43" width="0.254" layer="16"/>
 <via x="22.225" y="11.43" extent="1-16" drill="0.35"/>
-<wire x1="20.9" y1="11.43" x2="22.225" y2="11.43" width="0.1524" layer="1"/>
-<wire x1="22.606" y1="11.049" x2="22.225" y2="11.43" width="0.1524" layer="1"/>
-<wire x1="22.606" y1="11.049" x2="22.606" y2="10.635" width="0.1524" layer="1"/>
-<wire x1="22.737" y1="16.125" x2="21" y2="16.125" width="0.1524" layer="1"/>
-<wire x1="22.86" y1="17.305" x2="22.86" y2="16.248" width="0.1524" layer="1"/>
+<wire x1="20.9" y1="11.43" x2="22.225" y2="11.43" width="0.254" layer="1"/>
+<wire x1="22.606" y1="11.049" x2="22.225" y2="11.43" width="0.254" layer="1"/>
+<wire x1="22.606" y1="11.049" x2="22.606" y2="10.635" width="0.254" layer="1"/>
+<wire x1="22.737" y1="16.125" x2="21" y2="16.125" width="0.254" layer="1"/>
+<wire x1="22.86" y1="17.305" x2="22.86" y2="16.248" width="0.254" layer="1"/>
 <wire x1="22.86" y1="16.248" x2="22.737" y2="16.125" width="0.1524" layer="1"/>
-<wire x1="23.368" y1="15.494" x2="22.86" y2="16.002" width="0.1524" layer="1"/>
-<wire x1="22.86" y1="16.002" x2="22.86" y2="16.248" width="0.1524" layer="1"/>
+<wire x1="23.368" y1="15.494" x2="22.86" y2="16.002" width="0.254" layer="1"/>
+<wire x1="22.86" y1="16.002" x2="22.86" y2="16.248" width="0.254" layer="1"/>
 <wire x1="39.37" y1="24.384" x2="39.37" y2="24.13" width="0" layer="19" extent="16-16"/>
 </signal>
@@
 <contactref element="Q2" pad="MOSI"/>
 <contactref element="U2" pad="15"/>
-<wire x1="20.05" y1="9.58" x2="20.05" y2="8.779" width="0.1524" layer="1"/>
+<wire x1="20.05" y1="9.58" x2="20.05" y2="8.779" width="0.254" layer="1"/>
 <via x="21.987" y="5.62" extent="1-16" drill="0.35"/>
-<wire x1="21.971" y1="6.858" x2="20.05" y2="8.779" width="0.1524" layer="1"/>
+<wire x1="21.971" y1="6.858" x2="20.05" y2="8.779" width="0.254" layer="1"/>
 <wire x1="21.987" y1="5.62" x2="21.971" y2="5.636" width="0.1524" layer="1"/>
-<wire x1="21.971" y1="5.636" x2="21.971" y2="6.858" width="0.1524" layer="1"/>
+<wire x1="21.971" y1="5.636" x2="21.971" y2="6.858" width="0.254" layer="1"/>
 </signal>
 <signal name="RST">
@@
 <contactref element="U2" pad="16"/>
 <via x="21.987" y="8.112" extent="1-16" drill="0.35"/>
-<wire x1="21.987" y1="8.112" x2="20.9" y2="9.199" width="0.1524" layer="1"/>
-<wire x1="20.9" y1="9.199" x2="20.9" y2="10.43" width="0.1524" layer="1"/>
+<wire x1="21.987" y1="8.112" x2="20.9" y2="9.199" width="0.254" layer="1"/>
+<wire x1="20.9" y1="9.199" x2="20.9" y2="10.43" width="0.254" layer="1"/>
 <wire x1="21.987" y1="8.62" x2="21.987" y2="8.112" width="0.1524" layer="16"/>
 </signal>
@@
 <contactref element="S1" pad="A2"/>
 <contactref element="U2" pad="20"/>
-<wire x1="21.59" y1="13.97" x2="21.297" y2="13.97" width="0.1524" layer="1"/>
-<wire x1="20.9" y1="12.43" x2="20.9" y2="13.573" width="0.1524" layer="1"/>
-<wire x1="21.297" y1="13.97" x2="20.9" y2="13.573" width="0.1524" layer="1"/>
+<wire x1="21.59" y1="13.97" x2="21.297" y2="13.97" width="0.254" layer="1"/>
+<wire x1="20.9" y1="12.43" x2="20.9" y2="13.573" width="0.254" layer="1"/>
+<wire x1="21.297" y1="13.97" x2="20.9" y2="13.573" width="0.254" layer="1"/>
 <via x="21.59" y="13.97" extent="1-16" drill="0.35"/>
 <wire x1="21.59" y1="13.97" x2="30.988" y2="13.97" width="0.254" layer="16"/>
@@
 <wire x1="43.688" y1="9.906" x2="43.688" y2="9.017" width="0.254" layer="16"/>
 <via x="43.688" y="9.017" extent="1-16" drill="0.35"/>
-<wire x1="43.688" y1="9.017" x2="42.672" y2="9.017" width="0.1524" layer="1"/>
-<wire x1="42.672" y1="9.017" x2="40.93" y2="10.759" width="0.1524" layer="1"/>
-<wire x1="40.93" y1="10.759" x2="40.93" y2="12.535" width="0.1524" layer="1"/>
+<wire x1="43.688" y1="9.017" x2="42.672" y2="9.017" width="0.254" layer="1"/>
+<wire x1="42.672" y1="9.017" x2="40.93" y2="10.759" width="0.254" layer="1"/>
+<wire x1="40.93" y1="10.759" x2="40.93" y2="12.535" width="0.254" layer="1"/>
 <wire x1="35.433" y1="11.43" x2="42.164" y2="11.43" width="0.254" layer="16"/>
-<wire x1="30.988" y1="13.97" x2="32.258" y2="15.24" width="0.1524" layer="1"/>
-<wire x1="32.258" y1="15.24" x2="34.163" y2="15.24" width="0.1524" layer="1"/>
+<wire x1="30.988" y1="13.97" x2="32.258" y2="15.24" width="0.254" layer="1"/>
+<wire x1="32.258" y1="15.24" x2="34.163" y2="15.24" width="0.254" layer="1"/>
 </signal>
 <signal name="SDO">
@@
 <wire x1="28.17" y1="20.32" x2="29.845" y2="20.32" width="0.4064" layer="1"/>
 <wire x1="29.845" y1="20.32" x2="32.79" y2="20.32" width="0.4064" layer="1"/>
-<wire x1="8.89" y1="20.32" x2="9.93" y2="20.32" width="0.4064" layer="1"/>
+<wire x1="9.93" y1="20.32" x2="8.89" y2="20.32" width="0.4064" layer="1"/>
 <wire x1="7.62" y1="20.8275" x2="8.3825" y2="20.8275" width="0.4064" layer="1"/>
 <wire x1="8.3825" y1="20.8275" x2="8.89" y2="20.32" width="0.4064" layer="1"/>
@@
 <wire x1="20.32" y1="1.27" x2="21.59" y2="2.54" width="0.254" layer="16"/>
 <wire x1="22.733" y1="2.54" x2="21.59" y2="2.54" width="0.254" layer="16"/>
-<wire x1="25.17" y1="5.08" x2="25.17" y2="3.58" width="0.1524" layer="1"/>
-<wire x1="25.17" y1="3.58" x2="24.13" y2="2.54" width="0.1524" layer="1"/>
-<wire x1="24.13" y1="2.54" x2="22.733" y2="2.54" width="0.1524" layer="1"/>
+<wire x1="25.17" y1="5.08" x2="25.17" y2="3.58" width="0.254" layer="1"/>
+<wire x1="25.17" y1="3.58" x2="24.13" y2="2.54" width="0.254" layer="1"/>
+<wire x1="24.13" y1="2.54" x2="22.733" y2="2.54" width="0.254" layer="1"/>
 </signal>
 <signal name="COL4">

Commit message: update
Parts:
- removed Q2: ISP, library:ISP
- added JP1: (no value), pinhead:1X04
- added R5: 0, Resistor:RESC1005X40
- U2: device library:MLF20-4X4 -> library:QFN20-.45MMPITCH
Connections:
- new net N$3: R5.1, U1.13
- net CLK: now also JP1.3; no longer Q2.CLK
- net GND: now also U2.21; no longer U2.TH
- net MISO: now also JP1.2; no longer Q2.MISO
- net MOSI: now also JP1.1; no longer Q2.MOSI
- net OE: now also R5.2, U2.12; no longer U1.13, U2.11
- net RST: now also JP1.4; no longer Q2.RST
- net STCP: now also U2.11; no longer U2.12
Routing:
- net RST: track 6.52 -> 33.3 mm
- net MISO: track 3.28 -> 25.0 mm
- net CLK: track 7.85 -> 28.4 mm
- net MOSI: track 4.76 -> 21.9 mm
- net BTN: track 34.5 -> 28.4 mm
- net N$3: track 0.00 -> 3.03 mm
- net OE: track 3.76 -> 1.42 mm
- net VCC: track 75.3 -> 77.6 mm
- net RR1: track 39.8 -> 39.1 mm
- net ROW2: track 18.9 -> 19.6 mm
- net STCP: track 3.77 -> 4.42 mm
