File: cad/schematic.sch (EAGLE design)
At the start: 28 parts, among them Q1 FC-255, Q2 ISP, U1 74HC595, U2 ATTINY2313, U3 PCA21125

Commit message: wip
Parts:
- added IMG2: SLOT, library:SLOT
Changed lines of the file:
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@@
 <part name="LED16" library="library" deviceset="LG-T67K" device="" value="M18"/>
 <part name="IMG1" library="library" deviceset="IMAGE" device=""/>
+<part name="IMG2" library="library" deviceset="SLOT" device=""/>
 </parts>
 <sheets>
@@
 </instance>
 <instance part="IMG1" gate="G$1" x="210.82" y="-10.16" smashed="yes"/>
+<instance part="IMG2" gate="G$1" x="203.2" y="-10.16" smashed="yes"/>
 </instances>
 <busses>

Commit message: update
Parts:
- removed Q2: ISP, library:ISP
- added JP1: (no value), pinhead:PINHD-1X4
- added R5: 0, Resistor:R_CHIP-0402(1005-METRIC)
- U2: device library:ATTINY2313AMLF20-4X4 -> library:ATTINY2313AQFN20-3X3
Connections:
- new net N$3: R5.1, U1.OE
- net CLK: now also JP1.3; no longer Q2.SCK
- net MISO: now also JP1.2; no longer Q2.MISO
- net MOSI: now also JP1.1; no longer Q2.MOSI
- net OE: now also R5.2, U2.PB2; no longer U1.OE, U2.PB1
- net RST: now also JP1.4; no longer Q2.RST
- net STCP: now also U2.PB1; no longer U2.PB2
Changed lines of the file:
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@@
 <?xml version="1.0" encoding="utf-8"?>
 <!DOCTYPE eagle SYSTEM "eagle.dtd">
-<eagle version="9.6.2">
+<eagle version="9.4.2">
 <drawing>
 <settings>
-<setting alwaysvectorfont="yes"/>
+<setting alwaysvectorfont="no"/>
 <setting verticaltext="up"/>
 </settings>
@@
 <layers>
 <layer number="1" name="Top" color="4" fill="1" visible="no" active="no"/>
+<layer number="2" name="Route2" color="1" fill="3" visible="no" active="no"/>
+<layer number="3" name="Route3" color="4" fill="3" visible="no" active="no"/>
+<layer number="4" name="Route4" color="1" fill="4" visible="no" active="no"/>
+<layer number="5" name="Route5" color="4" fill="4" visible="no" active="no"/>
+<layer number="6" name="Route6" color="1" fill="8" visible="no" active="no"/>
+<layer number="7" name="Route7" color="4" fill="8" visible="no" active="no"/>
+<layer number="8" name="Route8" color="1" fill="2" visible="no" active="no"/>
+<layer number="9" name="Route9" color="4" fill="2" visible="no" active="no"/>
+<layer number="10" name="Route10" color="1" fill="7" visible="no" active="no"/>
+<layer number="11" name="Route11" color="4" fill="7" visible="no" active="no"/>
+<layer number="12" name="Route12" color="1" fill="5" visible="no" active="no"/>
+<layer number="13" name="Route13" color="4" fill="5" visible="no" active="no"/>
+<layer number="14" name="Route14" color="1" fill="6" visible="no" active="no"/>
+<layer number="15" name="Route15" color="4" fill="6" visible="no" active="no"/>
 <layer number="16" name="Bottom" color="1" fill="1" visible="no" active="no"/>
 <layer number="17" name="Pads" color="2" fill="1" visible="no" active="no"/>
@@
 <parts>
 <part name="U1" library="library" deviceset="74HC595" device=""/>
-<part name="U2" library="library" deviceset="ATTINY2313A" device="MLF20-4X4" value="ATTINY2313"/>
+<part name="U2" library="library" deviceset="ATTINY2313A" device="QFN20-3X3" value="ATTINY2313"/>
 <part name="U3" library="library" deviceset="PCA21125" device=""/>
 <part name="Q1" library="library" deviceset="FC-255" device=""/>
@@
 <part name="U$14" library="Airquality_Sensor" library_urn="urn:adsk.eagle:library:16015176" deviceset="GND" device=""/>
 <part name="S1" library="SparkFun-Switches" library_urn="urn:adsk.eagle:library:535" deviceset="MOMENTARY-SWITCH-SPST" device="-SMD-6.2MM-TALL" package3d_urn="urn:adsk.eagle:package:40172/1" value=""/>
-<part name="Q2" library="library" deviceset="ISP" device=""/>
 <part name="U$15" library="Evllve PCB Array" library_urn="urn:adsk.eagle:library:14885710" deviceset="VCC" device=""/>
 <part name="R4" library="Resistor" library_urn="urn:adsk.eagle:library:16378527" deviceset="R" device="CHIP-0402(1005-METRIC)" package3d_urn="urn:adsk.eagle:package:16378568/1" technology="_"/>
@@
 <part name="IMG1" library="library" deviceset="IMAGE" device=""/>
 <part name="IMG2" library="library" deviceset="SLOT" device=""/>
+<part name="R5" library="Resistor" library_urn="urn:adsk.eagle:library:16378527" deviceset="R" device="CHIP-0402(1005-METRIC)" package3d_urn="urn:adsk.eagle:package:16378568/1" technology="_" value="0"/>
+<part name="JP1" library="pinhead" library_urn="urn:adsk.eagle:library:325" deviceset="PINHD-1X4" device="" package3d_urn="urn:adsk.eagle:package:22407/2"/>
 </parts>
 <sheets>
@@
 <attribute name="VALUE" x="58.928" y="106.68" size="1.778" layer="96" font="vector" rot="R90" align="top-center"/>
 </instance>
-<instance part="Q2" gate="G$1" x="104.14" y="106.68" smashed="yes">
-<attribute name="NAME" x="101.6" y="114.808" size="1.778" layer="95" font="vector"/>
-<attribute name="VALUE" x="101.6" y="99.314" size="1.778" layer="96" font="vector"/>
-</instance>
 <instance part="U$15" gate="G$1" x="58.42" y="116.84" smashed="yes">
 <attribute name="VALUE" x="55.88" y="114.3" size="1.778" layer="96" rot="R90"/>
@@
 <instance part="IMG1" gate="G$1" x="210.82" y="-10.16" smashed="yes"/>
 <instance part="IMG2" gate="G$1" x="203.2" y="-10.16" smashed="yes"/>
+<instance part="R5" gate="G$1" x="63.5" y="-10.16" smashed="yes">
+<attribute name="NAME" x="60.96" y="-7.62" size="1.778" layer="95"/>
+<attribute name="VALUE" x="60.96" y="-13.97" size="1.778" layer="96"/>
+</instance>
+<instance part="JP1" gate="A" x="106.68" y="106.68" smashed="yes">
+<attribute name="NAME" x="100.33" y="114.935" size="1.778" layer="95"/>
+<attribute name="VALUE" x="100.33" y="99.06" size="1.778" layer="96"/>
+</instance>
 </instances>
 <busses>
@@
 <net name="MOSI" class="0">
 <segment>
-<pinref part="Q2" gate="G$1" pin="MOSI"/>
-<wire x1="99.06" y1="104.14" x2="91.44" y2="104.14" width="0.1524" layer="91"/>
-<label x="91.44" y="104.14" size="1.778" layer="95"/>
-</segment>
-<segment>
 <pinref part="U2" gate="G$1" pin="PB5"/>
 <wire x1="96.52" y1="83.82" x2="106.68" y2="83.82" width="0.1524" layer="91"/>
 <label x="99.06" y="83.82" size="1.778" layer="95"/>
 </segment>
+<segment>
+<pinref part="JP1" gate="A" pin="1"/>
+<wire x1="104.14" y1="111.76" x2="93.98" y2="111.76" width="0.1524" layer="91"/>
+<label x="93.98" y="111.76" size="1.778" layer="95"/>
+</segment>
 </net>
 <net name="RST" class="0">
-<segment>
-<pinref part="Q2" gate="G$1" pin="RST"/>
-<wire x1="99.06" y1="106.68" x2="91.44" y2="106.68" width="0.1524" layer="91"/>
-<label x="91.44" y="106.68" size="1.778" layer="95"/>
-</segment>
 <segment>
 <pinref part="U2" gate="G$1" pin="RESET"/>
@@
 <label x="58.42" y="63.5" size="1.778" layer="95"/>
 </segment>
+<segment>
+<pinref part="JP1" gate="A" pin="4"/>
+<wire x1="104.14" y1="104.14" x2="93.98" y2="104.14" width="0.1524" layer="91"/>
+<label x="93.98" y="104.14" size="1.778" layer="95"/>
+</segment>
 </net>
 <net name="CLK" class="0">
-<segment>
-<pinref part="Q2" gate="G$1" pin="SCK"/>
-<wire x1="99.06" y1="109.22" x2="91.44" y2="109.22" width="0.1524" layer="91"/>
-<label x="91.44" y="109.22" size="1.778" layer="95"/>
-</segment>
 <segment>
 <pinref part="U2" gate="G$1" pin="PB7"/>
@@
 <label x="99.06" y="88.9" size="1.778" layer="95"/>
 </segment>
+<segment>
+<pinref part="JP1" gate="A" pin="3"/>
+<wire x1="104.14" y1="106.68" x2="93.98" y2="106.68" width="0.1524" layer="91"/>
+<label x="93.98" y="106.68" size="1.778" layer="95"/>
+</segment>
 </net>
 <net name="MISO" class="0">
-<segment>
-<pinref part="Q2" gate="G$1" pin="MISO"/>
-<wire x1="99.06" y1="111.76" x2="91.44" y2="111.76" width="0.1524" layer="91"/>
-<label x="91.44" y="111.76" size="1.778" layer="95"/>
-</segment>
 <segment>
 <pinref part="U2" gate="G$1" pin="PB6"/>
@@
 <label x="99.06" y="86.36" size="1.778" layer="95"/>
 </segment>
+<segment>
+<pinref part="JP1" gate="A" pin="2"/>
+<wire x1="104.14" y1="109.22" x2="93.98" y2="109.22" width="0.1524" layer="91"/>
+<label x="93.98" y="109.22" size="1.778" layer="95"/>
+</segment>
 </net>
 <net name="INT" class="0">
@@
 </segment>
 <segment>
+<pinref part="U2" gate="G$1" pin="PB1"/>
+<wire x1="96.52" y1="73.66" x2="106.68" y2="73.66" width="0.1524" layer="91"/>
+<label x="99.06" y="73.66" size="1.778" layer="95"/>
+<label x="99.06" y="73.66" size="1.778" layer="95"/>
+</segment>
+</net>
+<net name="OE" class="0">
+<segment>
 <pinref part="U2" gate="G$1" pin="PB2"/>
 <wire x1="96.52" y1="76.2" x2="106.68" y2="76.2" width="0.1524" layer="91"/>
 <label x="99.06" y="76.2" size="1.778" layer="95"/>
 </segment>
-</net>
-<net name="OE" class="0">
-<segment>
-<pinref part="U1" gate="G$1" pin="OE"/>
-<wire x1="55.88" y1="-5.08" x2="55.88" y2="-12.7" width="0.1524" layer="91"/>
-<label x="55.88" y="-10.16" size="1.778" layer="95" rot="R90"/>
-</segment>
-<segment>
-<pinref part="U2" gate="G$1" pin="PB1"/>
-<wire x1="96.52" y1="73.66" x2="106.68" y2="73.66" width="0.1524" layer="91"/>
-<label x="99.06" y="73.66" size="1.778" layer="95"/>
+<segment>
+<pinref part="R5" gate="G$1" pin="2"/>
+<wire x1="68.58" y1="-10.16" x2="76.2" y2="-10.16" width="0.1524" layer="91"/>
+<label x="71.12" y="-10.16" size="1.778" layer="95"/>
 </segment>
 </net>
@@
 </segment>
 </net>
+<net name="N$3" class="0">
+<segment>
+<pinref part="R5" gate="G$1" pin="1"/>
+<pinref part="U1" gate="G$1" pin="OE"/>
+<wire x1="58.42" y1="-10.16" x2="55.88" y2="-10.16" width="0.1524" layer="91"/>
+<wire x1="55.88" y1="-10.16" x2="55.88" y2="-5.08" width="0.1524" layer="91"/>
+</segment>
+</net>
